File: hardware/schematics/schematics.sch (KiCad schematic (older format))
At the start: 26 parts, among them J1 Jack-DC, J2 Conn_01x20, J3 Conn_01x20, Q1 IRLD110PBF, U1 ESP32-DevKitC, U2 L7805, U3 MAX6921AUI+

Commit message: Wiring fixed
Parts:
- Q1: footprint Package_DIP:DIP-4_W7.62mm -> Package_DIP:Vishay_HVM-DIP-3_W7.62mm
Connections:
- net DIN: now also U1.J3_2 (GPIO23(SPI_MOSI)); no longer U1.J3_8 (GPIO19(SPI_MISO))
- net GND: now also J2.19 (Pin_19), J2.2 (Pin_2); no longer J2.1 (Pin_1), J2.20 (Pin_20)
- net O_0: now also J2.3 (Pin_3); no longer J2.18 (Pin_18)
- net O_1: now also J2.5 (Pin_5); no longer J2.16 (Pin_16)
- net O_10: now also J2.12 (Pin_12); no longer J2.9 (Pin_9)
- net O_11: now also J2.14 (Pin_14); no longer J2.7 (Pin_7)
- net O_12: now also J2.16 (Pin_16); no longer J2.5 (Pin_5)
- net O_13: now also J2.18 (Pin_18); no longer J2.3 (Pin_3)
- net O_16: now also J2.4 (Pin_4); no longer J2.17 (Pin_17)
- net O_17: now also J2.6 (Pin_6); no longer J2.15 (Pin_15)
- net O_18: now also J2.8 (Pin_8); no longer J2.13 (Pin_13)
- net O_19: now also J2.10 (Pin_10); no longer J2.11 (Pin_11)
- net O_2: now also J2.7 (Pin_7); no longer J2.14 (Pin_14)
- net O_3: now also J2.9 (Pin_9); no longer J2.12 (Pin_12)
- net O_4: now also J2.11 (Pin_11); no longer J2.10 (Pin_10)
- net O_5: now also J2.13 (Pin_13); no longer J2.8 (Pin_8)
- net O_6: now also J2.15 (Pin_15); no longer J2.6 (Pin_6)
- net O_7: now also J2.17 (Pin_17); no longer J2.4 (Pin_4)
- net O_8: now also J2.20 (Pin_20); no longer J2.2 (Pin_2)
- net dig_1: now also J3.6 (Pin_6); no longer J3.15 (Pin_15)
- net dig_2: now also J3.20 (Pin_20); no longer J3.1 (Pin_1)
- net dig_3: now also J3.8 (Pin_8); no longer J3.13 (Pin_13)
- net dig_4: now also J3.18 (Pin_18); no longer J3.3 (Pin_3)
- net dig_5: now also J3.10 (Pin_10); no longer J3.11 (Pin_11)
- net dig_6: now also J3.16 (Pin_16); no longer J3.5 (Pin_5)
- net dig_7: now also J3.14 (Pin_14); no longer J3.7 (Pin_7)
- net dig_8: now also J3.12 (Pin_12); no longer J3.9 (Pin_9)
- net dig_9: now also J3.4 (Pin_4); no longer J3.17 (Pin_17)
- net fil_g: now also J3.19 (Pin_19)
- net fil_v: now also J3.1 (Pin_1); no longer J3.20 (Pin_20)
- net seg_a: now also J3.9 (Pin_9); no longer J3.12 (Pin_12)
- net seg_b: now also J3.5 (Pin_5); no longer J3.16 (Pin_16)
- net seg_c: now also J3.15 (Pin_15); no longer J3.6 (Pin_6)
- net seg_d: now also J3.13 (Pin_13); no longer J3.8 (Pin_8)
- net seg_e: now also J3.17 (Pin_17); no longer J3.4 (Pin_4)
- net seg_f: now also J3.7 (Pin_7); no longer J3.14 (Pin_14)
- net seg_g: now also J3.3 (Pin_3); no longer J3.18 (Pin_18)
- net seg_h: now also J3.11 (Pin_11); no longer J3.10 (Pin_10)
- net at R3.1: now also J2.1 (Pin_1); no longer J2.19 (Pin_19)
- no-connect marks 31 -> 30
Other:
- moved on the sheet: R3
Changed lines of the file:
@@
 F 0 "Q1" H 5754 2096 50  0000 L CNN
 F 1 "IRLD110PBF" H 5754 2005 50  0000 L CNN
-F 2 "Package_DIP:DIP-4_W7.62mm" H 5750 2150 50  0001 C CNN
+F 2 "Package_DIP:Vishay_HVM-DIP-3_W7.62mm" H 5750 2150 50  0001 C CNN
 F 3 "~" H 5550 2050 50  0001 C CNN
 	1    5550 2050
@@
 $EndComp
 NoConn ~ 2950 5950
-NoConn ~ 3550 3800
 NoConn ~ 2800 5950
 NoConn ~ 2700 5950
@@
 Wire Wire Line
 	5750 5900 5750 6250
-$Comp
-L Connector_Generic:Conn_01x20 J3
-U 1 1 61196BBA
-P 7800 4850
-F 0 "J3" H 7718 3625 50  0000 C CNN
-F 1 "Conn_01x20" H 7718 3716 50  0000 C CNN
-F 2 "Connector_PinSocket_2.54mm:PinSocket_2x10_P2.54mm_Vertical" H 7800 4850 50  0001 C CNN
-F 3 "~" H 7800 4850 50  0001 C CNN
-	1    7800 4850
-	-1   0    0    1
-$EndComp
 $Comp
 L power:GND #PWR012
@@
 L power:VCC #PWR020
 U 1 1 6117890B
-P 6850 5200
-F 0 "#PWR020" H 6850 5050 50  0001 C CNN
-F 1 "VCC" H 6865 5373 50  0000 C CNN
-F 2 "" H 6850 5200 50  0001 C CNN
-F 3 "" H 6850 5200 50  0001 C CNN
-	1    6850 5200
+P 6850 3400
+F 0 "#PWR020" H 6850 3250 50  0001 C CNN
+F 1 "VCC" H 6865 3573 50  0000 C CNN
+F 2 "" H 6850 3400 50  0001 C CNN
+F 3 "" H 6850 3400 50  0001 C CNN
+	1    6850 3400
 	1    0    0    -1
 $EndComp
@@
 L Device:R R3
 U 1 1 610C9DA0
-P 6850 5450
-F 0 "R3" H 6750 5400 50  0000 C CNN
-F 1 "22" H 6750 5500 50  0000 C CNN
-F 2 "Resistor_THT:R_Axial_DIN0207_L6.3mm_D2.5mm_P10.16mm_Horizontal" V 6780 5450 50  0001 C CNN
-F 3 "~" H 6850 5450 50  0001 C CNN
-	1    6850 5450
+P 6850 3650
+F 0 "R3" H 6750 3600 50  0000 C CNN
+F 1 "22" H 6750 3700 50  0000 C CNN
+F 2 "Resistor_THT:R_Axial_DIN0207_L6.3mm_D2.5mm_P10.16mm_Horizontal" V 6780 3650 50  0001 C CNN
+F 3 "~" H 6850 3650 50  0001 C CNN
+	1    6850 3650
 	-1   0    0    1
 $EndComp
@@
 Text Label 3550 3600 0    50   ~ 0
 CLK
-Text Label 3550 3700 0    50   ~ 0
-DIN
 Text Label 3550 3900 0    50   ~ 0
 BLANK
@@
 	3550 3600 3850 3600
 Wire Wire Line
-	3550 3700 3850 3700
-Wire Wire Line
 	3550 3900 3850 3900
 Entry Wire Line
@@
 	3850 3600 3950 3500
 Entry Wire Line
-	3850 3700 3950 3600
+	3850 3800 3950 3700
 Entry Wire Line
 	3850 3900 3950 3800
@@
 	4650 3200 3950 3200
 Wire Wire Line
-	6850 5750 6850 6250
-Wire Wire Line
-	6850 5750 7250 5750
+	6850 5650 6850 6150
+Wire Wire Line
+	6850 5650 7250 5650
 Wire Wire Line
 	1200 1400 1200 1850
@@
 	3550 4150 4000 4150
 Wire Wire Line
-	6850 5200 6850 5300
-Wire Wire Line
-	6850 5650 7250 5650
-Wire Wire Line
-	6850 5600 6850 5650
+	6850 3400 6850 3500
+Wire Wire Line
+	6850 3850 7250 3850
+Wire Wire Line
+	6850 3800 6850 3850
 Wire Wire Line
 	1100 5150 1650 5150
@@
 Text Label 6450 3950 0    50   ~ 0
 O_1
-Text Label 7250 5350 2    50   ~ 0
+Text Label 7250 4250 2    50   ~ 0
 O_1
 Text Label 6450 4050 0    50   ~ 0
@@
 Text Label 6450 4350 0    50   ~ 0
 O_5
-Text Label 7250 5150 2    50   ~ 0
+Text Label 7250 4450 2    50   ~ 0
 O_2
-Text Label 7250 4950 2    50   ~ 0
+Text Label 7250 4650 2    50   ~ 0
 O_3
-Text Label 7250 4750 2    50   ~ 0
+Text Label 7250 4850 2    50   ~ 0
 O_4
-Text Label 7250 4550 2    50   ~ 0
+Text Label 7250 5050 2    50   ~ 0
 O_5
 Text Label 6450 3850 0    50   ~ 0
 O_0
-Text Label 7250 5550 2    50   ~ 0
+Text Label 7250 4050 2    50   ~ 0
 O_0
 Text Label 6450 4450 0    50   ~ 0
@@
 Text Label 6450 5750 0    50   ~ 0
 O_19
-Text Label 7250 4350 2    50   ~ 0
+Text Label 7250 5250 2    50   ~ 0
 O_6
-Text Label 7250 4150 2    50   ~ 0
-O_7
-Text Label 7250 3950 2    50   ~ 0
+Text Label 7600 6200 2    50   ~ 0
 O_8
 Text Label 6450 5650 0    50   ~ 0
@@
 Text Label 6450 5450 0    50   ~ 0
 O_16
-Text Label 7250 4850 2    50   ~ 0
+Text Label 7250 4750 2    50   ~ 0
 O_19
-Text Label 7250 5050 2    50   ~ 0
+Text Label 7250 4550 2    50   ~ 0
 O_18
-Text Label 7250 5250 2    50   ~ 0
+Text Label 7250 4350 2    50   ~ 0
 O_17
-Text Label 7250 5450 2    50   ~ 0
+Text Label 7250 4150 2    50   ~ 0
 O_16
 Text Label 6450 5150 0    50   ~ 0
@@
 Text Label 6450 4950 0    50   ~ 0
 O_11
-Text Label 7250 4650 2    50   ~ 0
+Text Label 7250 4950 2    50   ~ 0
 O_10
-Text Label 7250 4450 2    50   ~ 0
+Text Label 7250 5150 2    50   ~ 0
 O_11
-Text Label 7250 4250 2    50   ~ 0
+Text Label 7250 5350 2    50   ~ 0
 O_12
-Text Label 7250 4050 2    50   ~ 0
-O_13
 NoConn ~ 6450 4750
 NoConn ~ 6450 5250
@@
 L power:GND #PWR021
 U 1 1 6117ABA5
-P 6850 6250
-F 0 "#PWR021" H 6850 6000 50  0001 C CNN
-F 1 "GND" H 6855 6077 50  0000 C CNN
-F 2 "" H 6850 6250 50  0001 C CNN
-F 3 "" H 6850 6250 50  0001 C CNN
-	1    6850 6250
+P 6850 6150
+F 0 "#PWR021" H 6850 5900 50  0001 C CNN
+F 1 "GND" H 6855 5977 50  0000 C CNN
+F 2 "" H 6850 6150 50  0001 C CNN
+F 3 "" H 6850 6150 50  0001 C CNN
+	1    6850 6150
 	1    0    0    -1
 $EndComp
@@
 Text Label 8050 5750 0    50   ~ 0
 dig_2
-$Comp
-L power:GND #PWR019
-U 1 1 6120D033
-P 6850 3950
-F 0 "#PWR019" H 6850 3700 50  0001 C CNN
-F 1 "GND" H 6855 3777 50  0000 C CNN
-F 2 "" H 6850 3950 50  0001 C CNN
-F 3 "" H 6850 3950 50  0001 C CNN
-	1    6850 3950
-	1    0    0    -1
-$EndComp
-Wire Wire Line
-	7250 3850 6850 3850
-Wire Wire Line
-	6850 3850 6850 3950
 Text Label 8050 5650 0    50   ~ 0
 fil_g
-NoConn ~ 8000 3950
 Text Label 8050 4850 0    50   ~ 0
 seg_h
@@
 Wire Wire Line
 	10800 5600 10900 5600
+Text Label 8050 3950 0    50   ~ 0
+fil_g
+Wire Wire Line
+	8000 3950 8350 3950
+Entry Wire Line
+	8350 3950 8450 3850
+Wire Wire Line
+	3550 3800 3850 3800
+Text Label 3550 3800 0    50   ~ 0
+DIN
+NoConn ~ 3550 3700
+Wire Wire Line
+	6850 3950 6850 4450
+Wire Wire Line
+	6850 3950 7250 3950
+$Comp
+L power:GND #PWR0101
+U 1 1 615408DC
+P 6850 4450
+F 0 "#PWR0101" H 6850 4200 50  0001 C CNN
+F 1 "GND" H 6855 4277 50  0000 C CNN
+F 2 "" H 6850 4450 50  0001 C CNN
+F 3 "" H 6850 4450 50  0001 C CNN
+	1    6850 4450
+	1    0    0    -1
+$EndComp
+Text Label 7250 5750 2    50   ~ 0
+O_8
+Text Label 7250 5450 2    50   ~ 0
+O_7
+Text Label 7250 5550 2    50   ~ 0
+O_13
 Wire Bus Line
 	4650 3200 4650 4900
@@
 	3950 3200 3950 3800
 Wire Bus Line
+	8450 3500 8450 5650
+Wire Bus Line
 	8900 3500 8900 5000
 Wire Bus Line
 	11000 3500 11000 5500
-Wire Bus Line
-	8450 3500 8450 5650
+$Comp
+L Connector_Generic:Conn_01x20 J3
+U 1 1 61196BBA
+P 7800 4750
+F 0 "J3" H 7718 3525 50  0000 C CNN
+F 1 "Conn_01x20" H 7718 3616 50  0000 C CNN
+F 2 "Connector_PinSocket_2.54mm:PinSocket_2x10_P2.54mm_Vertical" H 7800 4750 50  0001 C CNN
+F 3 "~" H 7800 4750 50  0001 C CNN
+	1    7800 4750
+	-1   0    0    -1
+$EndComp
 $EndSCHEMATC

Commit message: Revision 2 of PCB, hopefully without workarounds
Parts:
- J2, J3: footprint Connector_PinSocket_2.54mm:PinSocket_2x10_P2.54mm_Vertical -> Connector_IDC:IDC-Header_2x10_P2.54mm_Vertical
- U2: footprint Package_TO_SOT_THT:TO-220-3_Vertical -> callisto:L7805_with_heatsink
- U3: value MAX6921AUI+ -> MAX6921AWI+; footprint Package_SO:TSSOP-28_4.4x9.7mm_P0.65mm -> Package_SO:SOIC-28W_7.5x17.9mm_P1.27mm; symbol callisto_lib:MAX6921AUI+ -> callisto_lib:MAX6921AWI+
Connections:
- net BLANK: now also U3.13 (BLANK); no longer U3.20 (BLANK)
- net CLK: now also U3.15 (CLK); no longer U3.22 (CLK)
- net DIN: now also U3.27 (DIN); no longer U3.6 (DIN)
- net GND: now also J2.1 (Pin_1), J2.20 (Pin_20), U3.14 (GND); no longer J2.19 (Pin_19), J2.2 (Pin_2), U3.21 (GND)
- net LOAD: now also U3.16 (LOAD); no longer U3.23 (LOAD)
- net O_0: now also J2.4 (Pin_4), U3.26 (OUT0); no longer J2.3 (Pin_3), U3.5 (OUT0)
- net O_1: now also J2.6 (Pin_6), U3.25 (OUT1); no longer J2.5 (Pin_5), U3.4 (OUT1)
- net O_11: now also J2.19 (Pin_19), U3.11 (OUT11); no longer J2.14 (Pin_14), U3.18 (OUT11)
- net O_12: now also J2.17 (Pin_17), U3.10 (OUT12); no longer J2.16 (Pin_16), U3.17 (OUT12)
- net O_13: now also J2.15 (Pin_15), U3.9 (OUT13); no longer J2.18 (Pin_18), U3.16 (OUT13)
- net O_16: now also J2.9 (Pin_9), U3.6 (OUT16); no longer J2.4 (Pin_4), U3.13 (OUT16)
- net O_17: now also J2.7 (Pin_7), U3.5 (OUT17); no longer J2.6 (Pin_6), U3.12 (OUT17)
- net O_18: now also J2.5 (Pin_5), U3.4 (OUT18); no longer J2.8 (Pin_8), U3.11 (OUT18)
- net O_19: now also J2.3 (Pin_3), U3.3 (OUT19); no longer J2.10 (Pin_10), U3.10 (OUT19)
- net O_2: now also J2.8 (Pin_8), U3.24 (OUT2); no longer J2.7 (Pin_7), U3.3 (OUT2)
- net O_3: now also J2.10 (Pin_10), U3.23 (OUT3); no longer J2.9 (Pin_9), U3.2 (OUT3)
- net O_4: now also J2.12 (Pin_12), U3.22 (OUT4); no longer J2.11 (Pin_11), U3.1 (OUT4)
- net O_5: now also J2.14 (Pin_14), U3.21 (OUT5); no longer J2.13 (Pin_13), U3.28 (OUT5)
- net O_6: now also J2.16 (Pin_16), U3.20 (OUT6); no longer J2.15 (Pin_15), U3.27 (OUT6)
- net O_7: now also J2.18 (Pin_18), U3.19 (OUT7); no longer J2.17 (Pin_17), U3.26 (OUT7)
- net VBB: now also U3.1 (VBB); no longer U3.8 (VBB)
- net VCC: now also U3.28 (VCC); no longer U3.7 (VCC)
- net dig_1: now also J3.5 (Pin_5); no longer J3.6 (Pin_6)
- net dig_2: now also J3.19 (Pin_19); no longer J3.20 (Pin_20)
- net dig_3: now also J3.7 (Pin_7); no longer J3.8 (Pin_8)
- net dig_4: now also J3.17 (Pin_17); no longer J3.18 (Pin_18)
- net dig_5: now also J3.9 (Pin_9); no longer J3.10 (Pin_10)
- net dig_6: now also J3.15 (Pin_15); no longer J3.16 (Pin_16)
- net dig_7: now also J3.13 (Pin_13); no longer J3.14 (Pin_14)
- net dig_8: now also J3.11 (Pin_11); no longer J3.12 (Pin_12)
- net dig_9: now also J3.3 (Pin_3); no longer J3.4 (Pin_4)
- net fil_g: now also J3.1 (Pin_1), J3.20 (Pin_20); no longer J3.19 (Pin_19), J3.2 (Pin_2)
- net fil_v: now also J3.2 (Pin_2); no longer J3.1 (Pin_1)
- net seg_a: now also J3.10 (Pin_10); no longer J3.9 (Pin_9)
- net seg_b: now also J3.6 (Pin_6); no longer J3.5 (Pin_5)
- net seg_c: now also J3.16 (Pin_16); no longer J3.15 (Pin_15)
- net seg_d: now also J3.14 (Pin_14); no longer J3.13 (Pin_13)
- net seg_e: now also J3.18 (Pin_18); no longer J3.17 (Pin_17)
- net seg_f: now also J3.8 (Pin_8); no longer J3.7 (Pin_7)
- net seg_g: now also J3.4 (Pin_4); no longer J3.3 (Pin_3)
- net seg_h: now also J3.12 (Pin_12); no longer J3.11 (Pin_11)
- net at R3.1: now also J2.2 (Pin_2); no longer J2.1 (Pin_1)
- removed net O_10: J2.12 (Pin_12), U3.19 (OUT10)
- removed net O_8: J2.20 (Pin_20), U3.25 (OUT8)
- new net DOUT: U3.2 (DOUT)
- new net O_14: J2.13 (Pin_13), U3.8 (OUT14)
- new net O_15: J2.11 (Pin_11), U3.7 (OUT15)
Other:
- moved on the sheet: R3
Changed lines of the file:
@@
 F 0 "U2" H 2800 1442 50  0000 C CNN
 F 1 "L7805" H 2800 1350 50  0000 C CNN
-F 2 "Package_TO_SOT_THT:TO-220-3_Vertical" H 2825 1050 50  0001 L CIN
+F 2 "callisto:L7805_with_heatsink" H 2825 1050 50  0001 L CIN
 F 3 "http://www.st.com/content/ccc/resource/technical/document/datasheet/41/4f/b3/b0/12/d4/47/88/CD00000444.pdf/files/CD00000444.pdf/jcr:content/translations/en.CD00000444.pdf" H 2800 1150 50  0001 C CNN
 	1    2800 1200
@@
 F 0 "J2" H 7450 5900 50  0000 C CNN
 F 1 "Conn_01x20" H 7450 5800 50  0000 C CNN
-F 2 "Connector_PinSocket_2.54mm:PinSocket_2x10_P2.54mm_Vertical" H 7450 4750 50  0001 C CNN
+F 2 "Connector_IDC:IDC-Header_2x10_P2.54mm_Vertical" H 7450 4750 50  0001 C CNN
 F 3 "~" H 7450 4750 50  0001 C CNN
 	1    7450 4750
@@
 L power:VCC #PWR020
 U 1 1 6117890B
-P 6850 3400
-F 0 "#PWR020" H 6850 3250 50  0001 C CNN
-F 1 "VCC" H 6865 3573 50  0000 C CNN
-F 2 "" H 6850 3400 50  0001 C CNN
-F 3 "" H 6850 3400 50  0001 C CNN
-	1    6850 3400
+P 6850 3350
+F 0 "#PWR020" H 6850 3200 50  0001 C CNN
+F 1 "VCC" H 6865 3523 50  0000 C CNN
+F 2 "" H 6850 3350 50  0001 C CNN
+F 3 "" H 6850 3350 50  0001 C CNN
+	1    6850 3350
 	1    0    0    -1
 $EndComp
@@
 L Device:R R3
 U 1 1 610C9DA0
-P 6850 3650
-F 0 "R3" H 6750 3600 50  0000 C CNN
-F 1 "22" H 6750 3700 50  0000 C CNN
-F 2 "Resistor_THT:R_Axial_DIN0207_L6.3mm_D2.5mm_P10.16mm_Horizontal" V 6780 3650 50  0001 C CNN
-F 3 "~" H 6850 3650 50  0001 C CNN
-	1    6850 3650
+P 6850 3600
+F 0 "R3" H 6750 3550 50  0000 C CNN
+F 1 "22" H 6750 3650 50  0000 C CNN
+F 2 "Resistor_THT:R_Axial_DIN0207_L6.3mm_D2.5mm_P10.16mm_Horizontal" V 6780 3600 50  0001 C CNN
+F 3 "~" H 6850 3600 50  0001 C CNN
+	1    6850 3600
 	-1   0    0    1
 $EndComp
@@
 	4650 3200 3950 3200
 Wire Wire Line
-	6850 5650 6850 6150
-Wire Wire Line
-	6850 5650 7250 5650
-Wire Wire Line
 	1200 1400 1200 1850
 Wire Wire Line
@@
 	-1   0    0    1
 $EndComp
-$Comp
-L callisto_lib:MAX6921AUI+ U3
-U 1 1 61130460
-P 5750 4800
-F 0 "U3" H 5200 5850 50  0000 C CNN
-F 1 "MAX6921AUI+" H 5200 5950 50  0000 C CNN
-F 2 "Package_SO:TSSOP-28_4.4x9.7mm_P0.65mm" H 5750 4800 50  0001 C CNN
-F 3 "" H 5750 4800 50  0001 C CNN
-	1    5750 4800
-	1    0    0    -1
-$EndComp
 Text Label 1600 6900 0    50   ~ 0
 BRIGHTNESS
@@
 	3550 4150 4000 4150
 Wire Wire Line
-	6850 3400 6850 3500
-Wire Wire Line
-	6850 3850 7250 3850
-Wire Wire Line
-	6850 3800 6850 3850
+	6850 3350 6850 3450
+Wire Wire Line
+	6850 3950 7250 3950
+Wire Wire Line
+	6850 3750 6850 3950
 Wire Wire Line
 	1100 5150 1650 5150
@@
 NoConn ~ 3550 4550
 Text Label 6450 3950 0    50   ~ 0
-O_1
-Text Label 7250 4250 2    50   ~ 0
 O_1
 Text Label 6450 4050 0    50   ~ 0
@@
 Text Label 6450 4350 0    50   ~ 0
 O_5
-Text Label 7250 4450 2    50   ~ 0
-O_2
-Text Label 7250 4650 2    50   ~ 0
-O_3
-Text Label 7250 4850 2    50   ~ 0
-O_4
-Text Label 7250 5050 2    50   ~ 0
-O_5
 Text Label 6450 3850 0    50   ~ 0
-O_0
-Text Label 7250 4050 2    50   ~ 0
 O_0
 Text Label 6450 4450 0    50   ~ 0
@@
 Text Label 6450 4550 0    50   ~ 0
 O_7
-Text Label 6450 4650 0    50   ~ 0
-O_8
 Text Label 6450 5750 0    50   ~ 0
 O_19
-Text Label 7250 5250 2    50   ~ 0
-O_6
-Text Label 7600 6200 2    50   ~ 0
-O_8
 Text Label 6450 5650 0    50   ~ 0
 O_18
@@
 Text Label 6450 5450 0    50   ~ 0
 O_16
-Text Label 7250 4750 2    50   ~ 0
-O_19
-Text Label 7250 4550 2    50   ~ 0
-O_18
-Text Label 7250 4350 2    50   ~ 0
-O_17
-Text Label 7250 4150 2    50   ~ 0
-O_16
 Text Label 6450 5150 0    50   ~ 0
 O_13
 Text Label 6450 5050 0    50   ~ 0
 O_12
-Text Label 6450 4850 0    50   ~ 0
-O_10
-Text Label 6450 4950 0    50   ~ 0
-O_11
-Text Label 7250 4950 2    50   ~ 0
-O_10
-Text Label 7250 5150 2    50   ~ 0
-O_11
-Text Label 7250 5350 2    50   ~ 0
-O_12
 NoConn ~ 6450 4750
-NoConn ~ 6450 5250
-NoConn ~ 6450 5350
-$Comp
-L power:GND #PWR021
-U 1 1 6117ABA5
-P 6850 6150
-F 0 "#PWR021" H 6850 5900 50  0001 C CNN
-F 1 "GND" H 6855 5977 50  0000 C CNN
-F 2 "" H 6850 6150 50  0001 C CNN
-F 3 "" H 6850 6150 50  0001 C CNN
-	1    6850 6150
-	1    0    0    -1
-$EndComp
 Wire Wire Line
 	8000 5750 8350 5750
 Entry Wire Line
 	8350 5750 8450 5650
-Text Label 8050 3850 0    50   ~ 0
+Text Label 8050 3950 0    50   ~ 0
 fil_v
+Text Label 8050 4050 0    50   ~ 0
+dig_9
+Text Label 8050 4250 0    50   ~ 0
+dig_1
+Text Label 8050 4450 0    50   ~ 0
+dig_3
+Text Label 8050 4650 0    50   ~ 0
+dig_5
+Text Label 8050 4850 0    50   ~ 0
+dig_8
+Text Label 8050 5050 0    50   ~ 0
+dig_7
+Text Label 8050 5250 0    50   ~ 0
+dig_6
+Text Label 8050 5450 0    50   ~ 0
+dig_4
+Text Label 8050 5650 0    50   ~ 0
+dig_2
+Text Label 8050 5750 0    50   ~ 0
+fil_g
+Text Label 8050 4950 0    50   ~ 0
+seg_h
+Text Label 8050 5150 0    50   ~ 0
+seg_d
+Text Label 8050 5350 0    50   ~ 0
+seg_c
+Text Label 8050 5550 0    50   ~ 0
+seg_e
+Text Label 8050 4750 0    50   ~ 0
+seg_a
+Text Label 8050 4550 0    50   ~ 0
+seg_f
+Text Label 8050 4350 0    50   ~ 0
+seg_b
 Text Label 8050 4150 0    50   ~ 0
-dig_9
-Text Label 8050 4350 0    50   ~ 0
-dig_1
-Text Label 8050 4550 0    50   ~ 0
-dig_3
-Text Label 8050 4750 0    50   ~ 0
-dig_5
-Text Label 8050 4950 0    50   ~ 0
-dig_8
-Text Label 8050 5150 0    50   ~ 0
-dig_7
-Text Label 8050 5350 0    50   ~ 0
-dig_6
-Text Label 8050 5550 0    50   ~ 0
-dig_4
-Text Label 8050 5750 0    50   ~ 0
-dig_2
-Text Label 8050 5650 0    50   ~ 0
-fil_g
-Text Label 8050 4850 0    50   ~ 0
-seg_h
-Text Label 8050 5050 0    50   ~ 0
-seg_d
-Text Label 8050 5250 0    50   ~ 0
-seg_c
-Text Label 8050 5450 0    50   ~ 0
-seg_e
-Text Label 8050 4650 0    50   ~ 0
-seg_a
-Text Label 8050 4450 0    50   ~ 0
-seg_f
-Text Label 8050 4250 0    50   ~ 0
-seg_b
-Text Label 8050 4050 0    50   ~ 0
 seg_g
 $Comp
@@
 Wire Wire Line
 	10800 5600 10900 5600
-Text Label 8050 3950 0    50   ~ 0
+Text Label 8050 3850 0    50   ~ 0
 fil_g
 Wire Wire Line
@@
 DIN
 NoConn ~ 3550 3700
-Wire Wire Line
-	6850 3950 6850 4450
-Wire Wire Line
-	6850 3950 7250 3950
 $Comp
 L power:GND #PWR0101
 U 1 1 615408DC
-P 6850 4450
-F 0 "#PWR0101" H 6850 4200 50  0001 C CNN
-F 1 "GND" H 6855 4277 50  0000 C CNN
-F 2 "" H 6850 4450 50  0001 C CNN
-F 3 "" H 6850 4450 50  0001 C CNN
-	1    6850 4450
-	1    0    0    -1
-$EndComp
-Text Label 7250 5750 2    50   ~ 0
-O_8
+P 7250 3850
+F 0 "#PWR0101" H 7250 3600 50  0001 C CNN
+F 1 "GND" H 7255 3677 50  0000 C CNN
+F 2 "" H 7250 3850 50  0001 C CNN
+F 3 "" H 7250 3850 50  0001 C CNN
+	1    7250 3850
+	0    1    1    0
+$EndComp
+$Comp
+L Connector_Generic:Conn_01x20 J3
+U 1 1 61196BBA
+P 7800 4750
+F 0 "J3" H 7718 3525 50  0000 C CNN
+F 1 "Conn_01x20" H 7718 3616 50  0000 C CNN
+F 2 "Connector_IDC:IDC-Header_2x10_P2.54mm_Vertical" H 7800 4750 50  0001 C CNN
+F 3 "~" H 7800 4750 50  0001 C CNN
+	1    7800 4750
+	-1   0    0    -1
+$EndComp
+Wire Wire Line
+	6850 5750 7250 5750
+Wire Wire Line
+	6850 5750 6850 6150
+Text Label 7250 5250 2    50   ~ 0
+O_13
 Text Label 7250 5450 2    50   ~ 0
+O_12
+Text Label 7250 4850 2    50   ~ 0
+O_15
+Text Label 7250 5350 2    50   ~ 0
+O_6
+Text Label 7250 5050 2    50   ~ 0
+O_14
+Text Label 7250 5150 2    50   ~ 0
+O_5
+Text Label 7250 4650 2    50   ~ 0
+O_16
+Text Label 7250 4450 2    50   ~ 0
+O_17
+Text Label 7250 4250 2    50   ~ 0
+O_18
+Text Label 7250 4050 2    50   ~ 0
+O_19
+Text Label 7250 4150 2    50   ~ 0
+O_0
+Text Label 7250 4950 2    50   ~ 0
+O_4
+Text Label 7250 4750 2    50   ~ 0
+O_3
+Text Label 7250 4550 2    50   ~ 0
+O_2
+Text Label 7250 4350 2    50   ~ 0
+O_1
+Text Label 7250 5650 2    50   ~ 0
+O_11
+Text Label 7250 5550 2    50   ~ 0
 O_7
-Text Label 7250 5550 2    50   ~ 0
-O_13
+$Comp
+L power:GND #PWR021
+U 1 1 6117ABA5
+P 6850 6150
+F 0 "#PWR021" H 6850 5900 50  0001 C CNN
+F 1 "GND" H 6855 5977 50  0000 C CNN
+F 2 "" H 6850 6150 50  0001 C CNN
+F 3 "" H 6850 6150 50  0001 C CNN
+	1    6850 6150
+	1    0    0    -1
+$EndComp
+$Comp
+L callisto_lib:MAX6921AWI+ U3
+U 1 1 61130460
+P 5750 4800
+F 0 "U3" H 5200 5850 50  0000 C CNN
+F 1 "MAX6921AWI+" H 5200 5950 50  0000 C CNN
+F 2 "Package_SO:SOIC-28W_7.5x17.9mm_P1.27mm" H 5750 4800 50  0001 C CNN
+F 3 "" H 5750 4800 50  0001 C CNN
+	1    5750 4800
+	1    0    0    -1
+$EndComp
+Text Label 6450 5250 0    50   ~ 0
+O_14
+Text Label 6450 5350 0    50   ~ 0
+O_15
+Text Label 6450 4950 0    50   ~ 0
+O_11
+NoConn ~ 6450 4850
+NoConn ~ 6450 4650
+Text Label 5050 4900 2    50   ~ 0
+DOUT
 Wire Bus Line
 	4650 3200 4650 4900
@@
 	3950 3200 3950 3800
 Wire Bus Line
-	8450 3500 8450 5650
-Wire Bus Line
 	8900 3500 8900 5000
 Wire Bus Line
 	11000 3500 11000 5500
-$Comp
-L Connector_Generic:Conn_01x20 J3
-U 1 1 61196BBA
-P 7800 4750
-F 0 "J3" H 7718 3525 50  0000 C CNN
-F 1 "Conn_01x20" H 7718 3616 50  0000 C CNN
-F 2 "Connector_PinSocket_2.54mm:PinSocket_2x10_P2.54mm_Vertical" H 7800 4750 50  0001 C CNN
-F 3 "~" H 7800 4750 50  0001 C CNN
-	1    7800 4750
-	-1   0    0    -1
-$EndComp
+Wire Bus Line
+	8450 3500 8450 5650
 $EndSCHEMATC
